File: kicad/km11.kicad_pcb (KiCad board)
At the start: 2 copper layers, 131.7 x 214.1 mm, 5 parts, among them J1 CONN-DEC-DOUBLE

Commit message: Initial routed
Parts:
- removed J1: CONN-DEC-DOUBLE, DEC-FLIP-CHIP:CONN-DEC-DOUBLE
- added C1: 100nF, Capacitor_SMD:C_0805_2012Metric, F.Cu at (290.8, 257.8)
- added C10: 10uF, Capacitor_SMD:CP_Elec_8x5.4, F.Cu at (237.5, 260.9)
- added C11: 10uF, Capacitor_SMD:CP_Elec_8x5.4, F.Cu at (237.5, 248.2)
- added C2: 100nF, Capacitor_SMD:C_0805_2012Metric, F.Cu at (204.5, 257.8)
- added C3: 100nF, Capacitor_SMD:C_0805_2012Metric, F.Cu at (309.9, 274.3)
- added C4: 100nF, Capacitor_SMD:C_0805_2012Metric, F.Cu at (291.1, 274.3)
- added C5: 100nF, Capacitor_SMD:C_0805_2012Metric, F.Cu at (273.1, 274.3)
- added C6: 100nF, Capacitor_SMD:C_0805_2012Metric, F.Cu at (240.3, 274.3)
- added C7: 100nF, Capacitor_SMD:C_0805_2012Metric, F.Cu at (222.6, 274.3)
- added C8: 100uF, Capacitor_SMD:CP_Elec_6.3x7.7, F.Cu at (265.3, 274.3)
- added C9: 100nF, Capacitor_SMD:C_0805_2012Metric, F.Cu at (205.7, 274.6)
- added D1: PWRLED, LED_SMD:LED_1206_3216Metric_Pad1.42x1.75mm_HandSolder, F.Cu at (261.4, 245.1)
- added D2: +3V_LED, LED_SMD:LED_1206_3216Metric_Pad1.42x1.75mm_HandSolder, F.Cu at (248.7, 245.1)
- added J2: display_switches_hdr, Connector_PinHeader_2.54mm:PinHeader_2x10_P2.54mm_Vertical, F.Cu at (281.9, 256.5)
- added J3: pgm_hdr, Connector_PinHeader_2.54mm:PinHeader_1x03_P2.54mm_Vertical, F.Cu at (228.6, 255.3)
- added J9: DEC-FLIP-CHIP_CONN-DEC-DOUBLE, DEC-FLIP-CHIP:CONN-DEC-DOUBLE, F.Cu at (330.2, 304.8)
- added JP1: Jumper_2_Bridged, Jumper:SolderJumper-2_P1.3mm_Bridged_RoundedPad1.0x1.5mm, F.Cu at (287.6, 264.2)
- added Q1: BC547, Package_TO_SOT_THT:TO-92_Inline, F.Cu at (320.0, 261.6)
- added R1: 4.7k, Resistor_SMD:R_0805_2012Metric, F.Cu at (240.4, 281.9)
- added R10: 1K, Resistor_SMD:R_0805_2012Metric, F.Cu at (267.1, 245.1)
- added R11: 1K, Resistor_SMD:R_0805_2012Metric, F.Cu at (254.4, 245.1)
- added R2: 4.7k, Resistor_SMD:R_0805_2012Metric, F.Cu at (260.7, 281.9)
- added R4: 1K, Resistor_SMD:R_0805_2012Metric, F.Cu at (279.8, 264.2)
- added R5: 1K, Resistor_SMD:R_0805_2012Metric, F.Cu at (310.2, 252.7)
- added R6: 1K, Resistor_SMD:R_0805_2012Metric, F.Cu at (310.2, 257.8)
- added R7: 1K, Resistor_SMD:R_0805_2012Metric, F.Cu at (302.6, 247.7)
- added R8: 1K, Resistor_SMD:R_0805_2012Metric, F.Cu at (310.2, 247.7)
- added R9: 1K, Resistor_SMD:R_0805_2012Metric, F.Cu at (310.2, 262.9)
- added U1: ATtiny1616-S, Package_SO:SOIC-20W_7.5x12.8mm_P1.27mm, F.Cu at (215.9, 257.8)
- added U2: PCF8574T, Package_SO:SOIC-16W_7.5x10.3mm_P1.27mm, F.Cu at (281.3, 274.3)
- added U3: PCF8574T, Package_SO:SOIC-16W_7.5x10.3mm_P1.27mm, F.Cu at (299.7, 274.3)
- added U4: PCF8574T, Package_SO:SOIC-16W_7.5x10.3mm_P1.27mm, F.Cu at (318.1, 274.3)
- added U5: PCF8574T, Package_SO:SOIC-16W_7.5x10.3mm_P1.27mm, F.Cu at (248.9, 274.3)
- added U6: PCF8574T, Package_SO:SOIC-16W_7.5x10.3mm_P1.27mm, F.Cu at (231.1, 274.3)
- added U7: PCF8574T, Package_SO:SOIC-16W_7.5x10.3mm_P1.27mm, F.Cu at (214.6, 274.3)
- added U8: 74ACT00SC, Package_SO:SOIC-14W_7.5x9mm_P1.27mm, F.Cu at (298.4, 257.8)
- added U9: LD1117S33TR_SOT223, Package_TO_SOT_SMD:SOT-223-3_TabPin2, F.Cu at (249.6, 257.8)
- H1, H2, H3, H4: renamed from  
- moved H1 143.5 mm to (204.3, 238.8)
- moved H2 143.5 mm to (254.8, 238.8)
- moved H3 143.5 mm to (273.8, 238.8)
- moved H4 143.5 mm to (324.6, 238.8)
Routing:
- net GND: track 0.00 -> 484.3 mm, vias 0 -> 8
- net +5V: track 0.00 -> 450.4 mm, vias 0 -> 7
- net /SDA: track 0.00 -> 168.3 mm, vias 0 -> 5
- net /SCL: track 0.00 -> 160.8 mm, vias 0 -> 5
- net /BSR7_H: track 0.00 -> 103.2 mm, vias 0 -> 1
- net /BSR1_H: track 0.00 -> 96.2 mm, vias 0 -> 1
- net /BSR3_H: track 0.00 -> 94.3 mm, vias 0 -> 2
- net /BSR8_H_2: track 0.00 -> 74.3 mm, vias 0 -> 1
- net /BSR0_H: track 0.00 -> 73.4 mm, vias 0 -> 1
- net /PB2: track 0.00 -> 69.1 mm, vias 0 -> 1
- net /TIMEOUT_H: track 0.00 -> 67.9 mm
- net /MOSI: track 0.00 -> 65.6 mm, vias 0 -> 1
- net /PB3: track 0.00 -> 64.8 mm, vias 0 -> 2
- net /MISO: track 0.00 -> 61.0 mm, vias 0 -> 1
- net /SPI_SS: track 0.00 -> 60.1 mm, vias 0 -> 2
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Other:
- board size 131.7 x 214.1 mm -> 131.7 x 70.6 mm
- net class Default removed
- board text removed: "Usable board space"
