File: kicad/km1105.kicad_pcb (KiCad board)
At the start: 2 copper layers, 131.7 x 80 mm, 42 parts, among them J1 CONN-DEC-DOUBLE, J2 display_switches_hdr, J3 pgm_hdr, Q1 BC547, U1 ATtiny1616-S, U2 PCF8574T, U3 PCF8574T, U4 PCF8574T, U5 PCF8574T, U6 PCF8574T, U7 PCF8574T, U8 74ACT00SC, U9 LD1117S33TR_SOT223

Commit message: Small typo fixed; add more description in readme
Connections:
- net /MOSI renamed /LCD_SDA_MOSI
- net /PB2 renamed /LCD_DC
- net /PB3 renamed /LCD_RST
- net /SCK renamed /LCD_SCK
- net /SPI_SS renamed /LCD_CS

Commit message: Bugfixes and 3d printed box
Parts:
- U8: footprint Package_SO:SOIC-14W_7.5x9mm_P1.27mm -> Package_SO:SO-14_3.9x8.65mm_P1.27mm
Routing:
- net /s4_on: track 74.9 -> 77.1 mm
- net /s4_off: track 106.8 -> 109.0 mm
- net GND: track 447.8 -> 450.0 mm
- net Net-(R5-Pad1): track 32.4 -> 34.5 mm, vias 3 -> 2
- net /s3_on: track 85.7 -> 84.8 mm
- net +5V: track 405.2 -> 404.3 mm
- net Net-(JP1-A): track 19.8 -> 20.6 mm
