File: kicad/km1105/km1105.kicad_sch (KiCad schematic)
At the start: 41 parts, among them J1 CONN-DEC-DOUBLE, J2 display_switches_hdr, J3 pgm_hdr, Q1 BC547, U1 ATtiny1616-S, U2 PCF8574T, U3 PCF8574T, U4 PCF8574T, U5 PCF8574T, U6 PCF8574T, U7 PCF8574T, U8 74ACT00SC, U9 LD1117S33TR_SOT223

Commit message: Update the display board
Parts:
- added C12: 100nF, Capacitor_SMD:C_0805_2012Metric, symbol Device:C
- added J4: la_01, Connector_PinHeader_2.54mm:PinHeader_2x20_P2.54mm_Vertical, symbol Connector_Generic:Conn_02x20_Odd_Even
- added J5: la_02, Connector_PinHeader_2.54mm:PinHeader_2x04_P2.54mm_Vertical, symbol Connector_Generic:Conn_02x04_Odd_Even
- added U10: SN74LVC245APW, Package_SO:TSSOP-20_4.4x6.5mm_P0.65mm, symbol Logic_LevelTranslator:SN74LVC245APW
- C10, C11: footprint Capacitor_SMD:CP_Elec_8x5.4 -> Capacitor_SMD:CP_Elec_4x4.5
Connections:
- net +3.3V: now also J2.2 (Pin_2), J2.4 (Pin_4), C12.1, U10.1 (DIR), U10.20 (VCC); no longer J2.15 (Pin_15), J2.17 (Pin_17)
- net +5V: no longer J2.2 (Pin_2)
- net BSR0_H: now also J4.32 (Pin_32)
- net BSR12_H: now also J4.4 (Pin_4)
- net BSR12_H_2: now also J5.3 (Pin_3)
- net BSR14_H: now also J4.6 (Pin_6)
- net BSR14_H_2: now also J5.5 (Pin_5)
- net BSR15_H: now also J4.8 (Pin_8)
- net BSR15_H_2: now also J5.7 (Pin_7)
- net BSR1_H: now also J4.30 (Pin_30)
- net BSR3_H: now also J4.28 (Pin_28)
- net BSR3_H_2: now also J5.4 (Pin_4)
- net BSR7_H: now also J4.26 (Pin_26)
- net BSR7_H_2: now also J5.2 (Pin_2)
- net BSR8_H: now also J4.2 (Pin_2)
- net BSR8_H_2: now also J5.1 (Pin_1)
- net B_MSYN_H: now also J4.11 (Pin_11)
- net B_SSYN_H: now also J4.9 (Pin_9)
- net C_H: now also J4.17 (Pin_17)
- net C_H_2: now also J4.10 (Pin_10)
- net GND: now also J2.10 (Pin_10), J2.12 (Pin_12), J2.14 (Pin_14), J2.16 (Pin_16), J2.18 (Pin_18), C12.2, J5.6 (Pin_6), J5.8 (Pin_8), U10.10 (GND), U10.19 (~{OE}), U10.7 (A6), U10.8 (A7), U10.9 (A8); no longer J2.19 (Pin_19)
- net ISR0_H: now also J4.39 (Pin_39)
- net ISR0_H_2: now also J4.40 (Pin_40)
- net ISR12_H: now also J4.27 (Pin_27)
- net ISR12_H_2: now also J4.20 (Pin_20)
- net ISR14_H: now also J4.29 (Pin_29)
- net ISR14_H_2: now also J4.22 (Pin_22)
- net ISR15_H: now also J4.31 (Pin_31)
- net ISR15_H_2: now also J4.24 (Pin_24)
- net ISR1_H: now also J4.37 (Pin_37)
- net ISR1_H_2: now also J4.38 (Pin_38)
- net ISR2_H: now also J4.1 (Pin_1)
- net ISR3_H: now also J4.35 (Pin_35)
- net ISR3_H_2: now also J4.36 (Pin_36)
- net ISR7_H: now also J4.33 (Pin_33)
- net ISR7_H_2: now also J4.34 (Pin_34)
- net ISR8_H: now also J4.25 (Pin_25)
- net ISR8_H_2: now also J4.18 (Pin_18)
- net LCD_CS: now also J2.19 (Pin_19), U10.14 (B5); no longer J2.10 (Pin_10), U1.2 (PA4)
- net LCD_DC: now also J2.17 (Pin_17), U10.15 (B4); no longer J2.12 (Pin_12), U1.9 (PB2)
- net LCD_RST: now also J2.15 (Pin_15), U10.16 (B3); no longer J2.14 (Pin_14), U1.8 (PB3)
- net LCD_SCK: now also J2.11 (Pin_11), U10.18 (B1); no longer J2.8 (Pin_8), U1.19 (PA3)
- net MISO: no longer J2.6 (Pin_6)
- net N_H: now also J4.23 (Pin_23)
- net N_H_2: now also J4.16 (Pin_16)
- net PB4: no longer J2.16 (Pin_16)
- net PB5: no longer J2.18 (Pin_18)
- net RW2_H: now also J4.7 (Pin_7)
- net TRAPS_H: now also J4.13 (Pin_13)
- net TST1_H: now also J4.5 (Pin_5)
- net TST2_H: now also J4.3 (Pin_3)
- net T_H: now also J4.15 (Pin_15)
- net V_H: now also J4.19 (Pin_19)
- net V_H_2: now also J4.12 (Pin_12)
- net Z_H: now also J4.21 (Pin_21)
- net Z_H_2: now also J4.14 (Pin_14)
- net s4_off: now also J2.6 (Pin_6), R9.2; no longer J2.11 (Pin_11), R7.2
- net s4_on: now also J2.8 (Pin_8), R7.2; no longer J2.13 (Pin_13), R9.2
- net LCD_SDA_MOSI renamed LCDU_MOSI
- net LCDU_MOSI: now also U10.3 (A2); no longer J2.4 (Pin_4)
- new net LCDU_CS: U1.2 (PA4), U10.6 (A5)
- new net LCDU_DC: U1.9 (PB2), U10.5 (A4)
- new net LCDU_RST: U1.8 (PB3), U10.4 (A3)
- new net LCDU_SCK: U1.19 (PA3), U10.2 (A1)
- new net LCD_MOSI: J2.13 (Pin_13), U10.17 (B2)
- no-connect marks 15 -> 40
Other:
- note added: "km1: msyn*, ssyn* bbsy*, but_ir*"
- note removed: "km1: msyn*, ssyn*, bbsy*, but_ir*"
- moved on the sheet: C10, C11, D1, D2, H1, H2, H3, H4, JP1, R10, R11, R7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
