File: kicad/km1105/km1105.kicad_sch (KiCad schematic)
At the start: 45 parts, among them J1 CONN-DEC-DOUBLE, J2 display_switches_hdr, J3 pgm_hdr, J4 la_01, J5 la_02, Q1 BC547, U1 ATtiny1616-S, U10 SN74LVC245APW, U2 PCF8574T, U3 PCF8574T, U4 PCF8574T, U5 PCF8574T, U6 PCF8574T, U7 PCF8574T, U8 74ACT00SC, U9 LD1117S33TR_SOT223

Commit message: Review against DEC KD11-B docs: fix ALU_S polarity, octal MPC, C0, AC LO
Checked both boards and the firmware against EK-KD11B-MM-001, the 11/05
print set (overlay drawings A-SS-5509081) and the KM11 W130/W131 prints;
the full record is in review.md. Every J1 pin and the whole lamp map in
km11-signals.txt verified correct. Corrections:

- ALU S3..S0 are dim-when-asserted on the KM-2 overlay, i.e. active low;
  signals.cpp now inverts U5 P4..P7 like it does the MPC.
- MPC is 8 bits and DEC quotes it in octal; it was shown as two decimal
  digits, which dropped the hundreds digit. Now 3 octal digits, and AMUX
  6 octal digits.
- The KM-2 bus cycle bits are C1 and C0 (00 DATI, 01 DATIP, 10 DATO,
  11 DATOB), not C1 and C2.
- KM11 pin B2 is BUS AC LO on the 11/05, not NO TIMEOUT: the display
  board switch and silkscreen are labelled AC LO (net name kept).
- Stale "runs at 3.3V" comments in kmmain.cpp and the Makefile: U1 is
  on +5V.

Co-Authored-By: Claude Fable 5.1 <noreply@anthropic.com>
Claude-Session: https://claude.ai/code/session_01MZqk7sLhEJokCQfByz3piz
Other:
- note added: "km2: c0*"
- note removed: "km2: c2*"
Changed lines of the file:
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@@
 		)
 	)
-	(text "km2: c2*"
+	(text "km2: c0*"
 		(exclude_from_sim no)
 		(at 155.956 105.918 0)
