File: kicad/kmdisp/kmdisp.kicad_pcb (KiCad board)
At the start: 2 copper layers, 59.4 x 38.5 mm, 8 parts, among them J1 lcd_conn, J2 display_switches_hdr, SW1 SW_Step, SW2 SW_SSYN, SW3 SW_ClkEna, SW4 SW_NoTimeout

Commit message: Fix documentation according to latest layout; fix edge connectors with chamfers
Parts:
- added G***: LOGO, LOGO, B.Cu at (86.1, 107.7)
Other:
- board size 59.4 x 38.5 mm -> 59.4 x 35.8 mm
- board text added: "CLK Enable"
- board text added: "Flatcable red -->"
- board text added: "No Timeout"
- board text added: "SSYN Enable"
- board text added: "Single Step"
- board text added: "lcd 128x160 1.8{dblquote}"
