File: kicad/kmdisp/kmdisp.kicad_pcb (KiCad board)
At the start: 2 copper layers, 59.4 x 35.8 mm, 9 parts, among them J1 lcd_conn, J2 display_switches_hdr, SW1 SW_Step, SW2 SW_SSYN, SW3 SW_ClkEna, SW4 SW_NoTimeout

Commit message: Review against DEC KD11-B docs: fix ALU_S polarity, octal MPC, C0, AC LO
Checked both boards and the firmware against EK-KD11B-MM-001, the 11/05
print set (overlay drawings A-SS-5509081) and the KM11 W130/W131 prints;
the full record is in review.md. Every J1 pin and the whole lamp map in
km11-signals.txt verified correct. Corrections:

- ALU S3..S0 are dim-when-asserted on the KM-2 overlay, i.e. active low;
  signals.cpp now inverts U5 P4..P7 like it does the MPC.
- MPC is 8 bits and DEC quotes it in octal; it was shown as two decimal
  digits, which dropped the hundreds digit. Now 3 octal digits, and AMUX
  6 octal digits.
- The KM-2 bus cycle bits are C1 and C0 (00 DATI, 01 DATIP, 10 DATO,
  11 DATOB), not C1 and C2.
- KM11 pin B2 is BUS AC LO on the 11/05, not NO TIMEOUT: the display
  board switch and silkscreen are labelled AC LO (net name kept).
- Stale "runs at 3.3V" comments in kmmain.cpp and the Makefile: U1 is
  on +5V.

Co-Authored-By: Claude Fable 5.1 <noreply@anthropic.com>
Claude-Session: https://claude.ai/code/session_01MZqk7sLhEJokCQfByz3piz
Parts:
- SW4: value SW_NoTimeout -> SW_AcLo
Other:
- board text added: "AC LO"
- board text removed: "No Timeout"
Changed lines of the file:
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@@
 			)
 		)
-		(property "Value" "SW_NoTimeout"
+		(property "Value" "SW_AcLo"
 			(at 0 -6.35 90)
 			(layer "F.Fab")
@@
 		)
 	)
-	(gr_text "No Timeout"
+	(gr_text "AC LO"
 		(at 110.74 104.79 90)
 		(layer "F.SilkS")
